Commit message: more changes

File: zebROS_ws/src/controller_node/urdf/2023_compbot.xacro (robot description, xacro)
@@ -3,9 +3,9 @@
     <link name="base_link"/>
     <!-- add important transforms for 2023 -->
-    <link name="intake"/>
-    <joint name="intake_joint" type="fixed">
+    <link name="front_bumper"/>
+    <joint name="front_bumper" type="fixed">
         <parent link="base_link"/>
-        <child link="intake"/>
-        <origin xyz="0.6561 0.0 0.210" rpy="0 0 0"/>
+        <child link="front_bumper"/>
+        <origin xyz="0.4445 0.0 0.0" rpy="0 0 0"/>
     </joint>
 </robot>
